Commit message: Diff_drive plugin in gazebo

File: diff_drive/urdf/ddrive.gazebo.xacro (robot description, xacro)
@@ -1,8 +1,7 @@
 <?xml version="1.0"?>
-<robot xmlns:xacro="http://www.ros.org/wiki/xacro" name="ddrive">
-  <gazebo reference="base_link">
+<robot>
+  <!-- <gazebo reference="base_link">
     <material>Gazebo/Blue</material>
   </gazebo>
-  <!-- Link1 -->
   <gazebo reference="right_wheel">
     <material>Gazebo/Orange</material>
@@ -13,7 +12,24 @@
   <gazebo reference="right_caster">
     <material>Gazebo/Red</material>
+    <mu1>0.0</mu1>
+    <mu2>0.0</mu2>
   </gazebo>
   <gazebo reference="left_caster">
     <material>Gazebo/Red</material>
+    <mu1>0.0</mu1>
+    <mu2>0.0</mu2>
+  </gazebo> -->
+  <gazebo>
+    <plugin
+      filename="libignition-gazebo-diff-drive-system.so"
+      name="ignition::gazebo::systems::DiffDrive">
+      <left_joint>base_link_to_left_wheel</left_joint>
+      <right_joint>base_link_to_right_wheel</right_joint>
+      <wheel_separation>0.8</wheel_separation>
+      <wheel_radius>0.3</wheel_radius>
+      <odom_publish_frequency>100</odom_publish_frequency>
+      <!-- <topic>/model/my_custom_model/cmd_vel</topic> -->
+      <!-- <topic>/cmd_vel</topic> -->
+    </plugin>
   </gazebo>
 </robot>

File: diff_drive/urdf/ddrive.urdf.xacro (robot description, xacro)
@@ -17,4 +17,5 @@
 <xacro:property name="body_mass"  value="${ros__parameters['body_mass']}" />
 <xacro:include filename="$(find diff_drive)/ddrive.gazebo.xacro" />
+<!-- <link name="world"/>  -->
 <material name = "red">
     <color rgba ="1 0 0 1" />
@@ -26,5 +27,4 @@
     <color rgba ="0 1 0 1" />
 </material>
-<!-- <link name="world"/>  -->
 <xacro:macro name="wheel_inertial" params="mass">
     <inertial>
@@ -87,16 +87,16 @@
         <xacro:caster_inertial mass="${caster_mass}"/>
     </link>
-    <!-- <joint name="base_link_to_${prefix}_caster" type="continuous">
+    <joint name="base_link_to_${prefix}_caster" type="continuous">
         <parent link="base_link"/>
         <child link="${prefix}_caster"/>
         <axis xyz="0 0 1"/>
         <origin rpy="0 1.57075 0" xyz="0 -${body_x/2 + caster_radius*2} ${reflect*(body_z/2 + caster_radius)}"/>
-    </joint> -->
-    <joint name="base_link_to_${prefix}_caster_turn" type="continuous">
+    </joint>
+    <!-- <joint name="base_link_to_${prefix}_caster_turn" type="continuous">
         <parent link="base_link"/>
         <child link="${prefix}_caster"/>
         <axis xyz="1 0 0"/>
         <origin rpy="0 1.57075 0" xyz="0 -${body_x/2 + caster_radius*2} ${reflect*(body_z/2 + caster_radius)}"/>
-    </joint>
+    </joint> -->
 </xacro:macro>
   <link name="base_link">

Commit message: Bridge works. Used teleop_key and it moves/flips.

File: diff_drive/urdf/ddrive.gazebo.xacro (robot description, xacro)
@@ -30,5 +30,5 @@
       <odom_publish_frequency>100</odom_publish_frequency>
       <!-- <topic>/model/my_custom_model/cmd_vel</topic> -->
-      <!-- <topic>/cmd_vel</topic> -->
+      <topic>/cmd_vel</topic>
     </plugin>
   </gazebo>

File: diff_drive/urdf/ddrive.urdf.xacro (robot description, xacro)
@@ -65,5 +65,5 @@
         <child link="${prefix}_wheel"/>
         <axis xyz="0 0 1"/>
-        <origin rpy="0 1.57075 0" xyz="${reflect*(body_x/2 + wheel_length/2)} ${body_x/2} 0"/>
+        <origin rpy="0 1.57075 0" xyz="${reflect*(body_x/2 + wheel_length/2)} ${body_x/2 - 0.2} 0"/>
     </joint>
 </xacro:macro>
@@ -91,5 +91,5 @@
         <child link="${prefix}_caster"/>
         <axis xyz="0 0 1"/>
-        <origin rpy="0 1.57075 0" xyz="0 -${body_x/2 + caster_radius*2} ${reflect*(body_z/2 + caster_radius)}"/>
+        <origin rpy="0 1.57075 0" xyz="0 -${body_x/2 - 0.1} ${reflect*(body_z/2 + caster_radius)}"/>
     </joint>
     <!-- <joint name="base_link_to_${prefix}_caster_turn" type="continuous">

Commit message: Added flip node and works

File: diff_drive/urdf/ddrive.gazebo.xacro (robot description, xacro)
@@ -9,15 +9,15 @@
   <gazebo reference="left_wheel">
     <material>Gazebo/Orange</material>
-  </gazebo>
+  </gazebo> -->
   <gazebo reference="right_caster">
-    <material>Gazebo/Red</material>
+    <!-- <material>Gazebo/Red</material> -->
     <mu1>0.0</mu1>
     <mu2>0.0</mu2>
   </gazebo>
   <gazebo reference="left_caster">
-    <material>Gazebo/Red</material>
+    <!-- <material>Gazebo/Red</material> -->
     <mu1>0.0</mu1>
     <mu2>0.0</mu2>
-  </gazebo> -->
+  </gazebo>
   <gazebo>
     <plugin

Commit message: Cleaned up code

File: diff_drive/urdf/ddrive.gazebo.xacro (robot description, xacro)
@@ -1,20 +1,9 @@
 <?xml version="1.0"?>
 <robot>
-  <!-- <gazebo reference="base_link">
-    <material>Gazebo/Blue</material>
-  </gazebo>
-  <gazebo reference="right_wheel">
-    <material>Gazebo/Orange</material>
-  </gazebo>
-  <gazebo reference="left_wheel">
-    <material>Gazebo/Orange</material>
-  </gazebo> -->
   <gazebo reference="right_caster">
-    <!-- <material>Gazebo/Red</material> -->
     <mu1>0.0</mu1>
     <mu2>0.0</mu2>
   </gazebo>
   <gazebo reference="left_caster">
-    <!-- <material>Gazebo/Red</material> -->
     <mu1>0.0</mu1>
     <mu2>0.0</mu2>
@@ -29,5 +18,4 @@
       <wheel_radius>0.3</wheel_radius>
       <odom_publish_frequency>100</odom_publish_frequency>
-      <!-- <topic>/model/my_custom_model/cmd_vel</topic> -->
       <topic>/cmd_vel</topic>
     </plugin>

File: diff_drive/urdf/ddrive.urdf.xacro (robot description, xacro)
@@ -17,5 +17,4 @@
 <xacro:property name="body_mass"  value="${ros__parameters['body_mass']}" />
 <xacro:include filename="$(find diff_drive)/ddrive.gazebo.xacro" />
-<!-- <link name="world"/>  -->
 <material name = "red">
     <color rgba ="1 0 0 1" />
@@ -50,6 +49,4 @@
             </geometry>
             <material name = "${color}" />
-            <!-- <origin xyz="0 0 -${leglen/2}" rpy="0 ${pi/2} 0"/> -->
-            <!-- <material name="white"/> -->
         </visual>
         <collision>
@@ -57,5 +54,4 @@
                 <cylinder length="${wheel_length}" radius="${wheel_radius}"/>
             </geometry>
-            <!-- <origin xyz="0 0 -${leglen/2}" rpy="0 ${pi/2} 0"/> -->
         </collision>
         <xacro:wheel_inertial mass="${wheel_mass}"/>
@@ -72,16 +68,12 @@
         <visual>
             <geometry>
-                <!-- <cylinder length="0.1" radius="0.1"/> -->
                 <sphere radius="${caster_radius}"/>
             </geometry>
-            <!-- <origin xyz="0 0 -${leglen/2}" rpy="0 ${pi/2} 0"/> -->
             <material name = "${color}" />
         </visual>
         <collision>
             <geometry>
-                <!-- <cylinder length="${caster_length}" radius="${caster_radius}"/> -->
                 <sphere radius="${caster_radius}"/>
             </geometry>
-            <!-- <origin xyz="0 0 -${leglen/2}" rpy="0 ${pi/2} 0"/> -->
         </collision>
         <xacro:caster_inertial mass="${caster_mass}"/>
@@ -93,10 +85,4 @@
         <origin rpy="0 1.57075 0" xyz="0 -${body_x/2 - 0.1} ${reflect*(body_z/2 + caster_radius)}"/>
     </joint>
-    <!-- <joint name="base_link_to_${prefix}_caster_turn" type="continuous">
-        <parent link="base_link"/>
-        <child link="${prefix}_caster"/>
-        <axis xyz="1 0 0"/>
-        <origin rpy="0 1.57075 0" xyz="0 -${body_x/2 + caster_radius*2} ${reflect*(body_z/2 + caster_radius)}"/>
-    </joint> -->
 </xacro:macro>
   <link name="base_link">

Commit message: Robot moves in RVIZ as in Gazebo

File: diff_drive/urdf/ddrive.gazebo.xacro (robot description, xacro)
@@ -19,4 +19,7 @@
       <odom_publish_frequency>100</odom_publish_frequency>
       <topic>/cmd_vel</topic>
+      <tf_topic>/tf</tf_topic>
+      <frame_id>/odom</frame_id>
+      <child_frame_id>/base_link</child_frame_id>
     </plugin>
   </gazebo>

File: diff_drive/urdf/ddrive.urdf.xacro (robot description, xacro)
@@ -68,5 +68,5 @@
         <child link="${prefix}_wheel"/>
         <axis xyz="0 0 1"/>
-        <origin rpy="0 1.57075 0" xyz="${reflect*(body_x/2 + wheel_length/2)} ${body_x/2 - 0.2} 0"/>
+        <origin rpy="1.57075 1.57075 0" xyz="${body_x/2 - 0.2} ${reflect*(body_x/2 + wheel_length/2)} 0"/>
     </joint>
 </xacro:macro>
@@ -90,5 +90,5 @@
         <child link="${prefix}_caster"/>
         <axis xyz="0 0 1"/>
-        <origin rpy="0 1.57075 0" xyz="0 -${body_x/2 - 0.1} ${reflect*(body_z/2 + caster_radius)}"/>
+        <origin rpy="0 1.57075 1.57075" xyz="-${body_x/2 - 0.1} 0 ${reflect*(body_z/2 + caster_radius)}"/>
     </joint>
 </xacro:macro>
@@ -99,4 +99,5 @@
       </geometry>
       <material name = "red" />
+       <origin rpy="0 0 1.57075" xyz="0 0 0"/>
     </visual>
     <collision>
@@ -104,4 +105,5 @@
         <box size="${body_x} ${body_y} ${body_z}"/>
       </geometry>
+      <origin rpy="0 0 1.57075" xyz="0 0 0"/>
     </collision>
     <xacro:body_inertial mass="${body_mass}"/>
