Commit message: Added macro to urdf. car in riviz done

File: diff_drive/urdf/ddrive.urdf.xacro (robot description, xacro)
@@ -8,91 +8,73 @@
 <xacro:property name="wheel_radius"  value="${ros__parameters['wheel_radius']}" />
 <xacro:property name="stem_lenght"  value="${platform_height-wheel_radius-wheel_radius-0.2-0.41-0.1}" />
-  <link name="Platform">
+<xacro:macro name="wheel" params="prefix reflect">
+    <link name="${prefix}_wheel">
+        <visual>
+            <geometry>
+                <cylinder length="0.1" radius="0.3"/>
+            </geometry>
+            <!-- <origin xyz="0 0 -${leglen/2}" rpy="0 ${pi/2} 0"/> -->
+            <!-- <material name="white"/> -->
+        </visual>
+        <collision>
+            <geometry>
+                <cylinder length="0.1" radius="0.3"/>
+            </geometry>
+            <!-- <origin xyz="0 0 -${leglen/2}" rpy="0 ${pi/2} 0"/> -->
+        </collision>
+        <!-- <xacro:default_inertial mass="10"/> -->
+    </link>
+    <joint name="base_link_to_${prefix}_wheel" type="continuous">
+        <parent link="base_link"/>
+        <child link="${prefix}_wheel"/>
+        <axis xyz="0 0 1"/>
+        <origin rpy="0 1.57075 0" xyz="${reflect*(0.8/2 + 0.1/2)} ${0.2/2 + stem_lenght/2} 0"/>
+    </joint>
+</xacro:macro>
+<xacro:macro name="caster" params="prefix reflect">
+    <link name="${prefix}_caster">
+        <visual>
+            <geometry>
+                <cylinder length="0.1" radius="0.1"/>
+            </geometry>
+            <!-- <origin xyz="0 0 -${leglen/2}" rpy="0 ${pi/2} 0"/> -->
+            <!-- <material name="white"/> -->
+        </visual>
+        <collision>
+            <geometry>
+                <cylinder length="0.1" radius="0.1"/>
+            </geometry>
+            <!-- <origin xyz="0 0 -${leglen/2}" rpy="0 ${pi/2} 0"/> -->
+        </collision>
+        <!-- <xacro:default_inertial mass="10"/> -->
+    </link>
+    <joint name="base_link_to_${prefix}_caster" type="continuous">
+        <parent link="base_link"/>
+        <child link="${prefix}_caster"/>
+        <axis xyz="0 0 1"/>
+        <origin rpy="0 1.57075 0" xyz="0 -${0.2/2 + stem_lenght/2 + 0.1} ${reflect*(0.2/2 + 0.1)}"/>
+    </joint>
+    <joint name="base_link_to_${prefix}_caster_turn" type="continuous">
+        <parent link="base_link"/>
+        <child link="${prefix}_caster"/>
+        <axis xyz="1 0 0"/>
+        <origin rpy="0 1.57075 0" xyz="0 -${0.2/2 + stem_lenght/2 + 0.1} ${reflect*(0.2/2 + 0.1)}"/>
+    </joint>
+</xacro:macro>
+  <link name="base_link">
     <visual>
       <geometry>
-        <cylinder length="0.1" radius="0.4"/>
-      </geometry>
-      <origin rpy="0 0 1.57075" xyz="0 0 0"/>
-    </visual>
-    <collision>
-      <geometry>
-        <cylinder length="0.1" radius="0.4"/>
-      </geometry>
-      <origin rpy="0 0 1.57075" xyz="0 0 0"/>
-    </collision>
-  </link>
-  <link name="Neck">
-    <visual>
-      <geometry>
-        <cylinder length="0.41" radius="0.05"/>
+        <box size="0.8 1.5 0.2"/>
       </geometry>
     </visual>
     <collision>
       <geometry>
-        <cylinder length="0.41" radius="0.05"/>
+        <box size="0.8 1.5 0.2"/>
       </geometry>
     </collision>
   </link>
-  <joint name="Neck_to_Platform" type="revolute">
-    <parent link="Neck"/>
-    <child link="Platform"/>
-    <origin xyz="0 0 ${0.1/2 + 0.41/2}"/>
-    <axis xyz="1 0 0"/>
-    <limit effort="1000.0" lower="-1.1" upper="1.1" velocity="0.5"/>
-  </joint>
-  <link name="base_link">
-    <visual>
-      <geometry>
-        <box size="0.6 0.4 0.2"/>
-      </geometry>
-    </visual>
-    <collision>
-      <geometry>
-        <box size="0.6 0.4 0.2"/>
-      </geometry>
-    </collision>
-  </link>
-  <joint name="base_link_to_Neck" type="fixed">
-    <parent link="base_link"/>
-    <child link="Neck"/>
-    <origin xyz="0 0 ${0.2/2 + 0.41/2}"/>
-  </joint>
-  <link name="stem">
-    <visual>
-      <geometry>
-        <cylinder length="${stem_lenght}" radius="0.1"/>
-      </geometry>
-    </visual>
-    <collision>
-      <geometry>
-        <cylinder length="${stem_lenght}" radius="0.1"/>
-      </geometry>
-    </collision>
-  </link>
-  <joint name="base_link_to_stem" type="continuous">
-    <parent link="base_link"/>
-    <child link="stem"/>
-    <axis xyz="0 0 -1"/>
-    <origin xyz="0 0 -${0.2/2 + stem_lenght/2}"/>
-  </joint>
-  <link name="wheel">
-    <visual>
-      <geometry>
-        <cylinder length="0.1" radius="${wheel_radius}"/>
-      </geometry>
-      <origin rpy="0 1.57075 0" xyz="0 0 0"/>
-    </visual>
-    <collision>
-      <geometry>
-        <cylinder length="0.1" radius="${wheel_radius}"/>
-      </geometry>
-      <origin rpy="0 1.57075 0" xyz="0 0 0"/>
-    </collision>
-  </link>
-  <joint name="stem_to_wheel" type="continuous">
-    <parent link="stem"/>
-    <child link="wheel"/>
-    <axis xyz="1 0 0"/>
-    <origin xyz="0 0 -${wheel_radius + (stem_lenght/2)}"/>
-  </joint>
+<xacro:wheel prefix="right" reflect="1" />
+<xacro:wheel prefix="left" reflect="-1" />
+<xacro:caster prefix="top" reflect="1" />
+<xacro:caster prefix="bottom" reflect="-1" />
 </robot>

Commit message: Have a world howing up without the robot

File: diff_drive/urdf/ddrive.urdf.xacro (robot description, xacro)
@@ -7,5 +7,30 @@
 <xacro:property name="platform_height"  value="${ros__parameters['platform_height']}" />
 <xacro:property name="wheel_radius"  value="${ros__parameters['wheel_radius']}" />
+<xacro:property name="wheel_length"  value="${ros__parameters['wheel_length']}" />
+<xacro:property name="wheel_mass"  value="${ros__parameters['wheel_mass']}" />
+<xacro:property name="caster_radius"  value="${ros__parameters['caster_radius']}" />
+<xacro:property name="caster_length"  value="${ros__parameters['caster_length']}" />
+<xacro:property name="caster_mass"  value="${ros__parameters['caster_mass']}" />
+<xacro:property name="body_x"  value="${ros__parameters['body_x']}" />
+<xacro:property name="body_y"  value="${ros__parameters['body_y']}" />
+<xacro:property name="body_z"  value="${ros__parameters['body_z']}" />
+<xacro:property name="body_mass"  value="${ros__parameters['body_mass']}" />
 <xacro:property name="stem_lenght"  value="${platform_height-wheel_radius-wheel_radius-0.2-0.41-0.1}" />
+<xacro:macro name="wheel_inertial" params="mass">
+    <inertial>
+            <mass value="${mass}" />
+            <inertia ixx="1e-3" ixy="0.0" ixz="0.0"
+                 iyy="1e-3" iyz="0.0"
+                 izz="1e-3" />
+    </inertial>
+</xacro:macro>
+<xacro:macro name="caster_inertial" params="mass">
+    <inertial>
+            <mass value="${mass}" />
+            <inertia ixx="1e-3" ixy="0.0" ixz="0.0"
+                 iyy="1e-3" iyz="0.0"
+                 izz="1e-3" />
+    </inertial>
+</xacro:macro>
 <xacro:macro name="wheel" params="prefix reflect">
     <link name="${prefix}_wheel">
@@ -19,9 +44,9 @@
         <collision>
             <geometry>
-                <cylinder length="0.1" radius="0.3"/>
+                <cylinder length="${wheel_length}" radius="${wheel_radius}"/>
             </geometry>
             <!-- <origin xyz="0 0 -${leglen/2}" rpy="0 ${pi/2} 0"/> -->
         </collision>
-        <!-- <xacro:default_inertial mass="10"/> -->
+        <xacro:wheel_inertial mass="${wheel_mass}"/>
     </link>
     <joint name="base_link_to_${prefix}_wheel" type="continuous">
@@ -29,5 +54,5 @@
         <child link="${prefix}_wheel"/>
         <axis xyz="0 0 1"/>
-        <origin rpy="0 1.57075 0" xyz="${reflect*(0.8/2 + 0.1/2)} ${0.2/2 + stem_lenght/2} 0"/>
+        <origin rpy="0 1.57075 0" xyz="${reflect*(body_x/2 + wheel_length/2)} ${body_x/2} 0"/>
     </joint>
 </xacro:macro>
@@ -39,13 +64,13 @@
             </geometry>
             <!-- <origin xyz="0 0 -${leglen/2}" rpy="0 ${pi/2} 0"/> -->
-            <!-- <material name="white"/> -->
+            <material name="white"/>
         </visual>
         <collision>
             <geometry>
-                <cylinder length="0.1" radius="0.1"/>
+                <cylinder length="${caster_length}" radius="${caster_radius}"/>
             </geometry>
             <!-- <origin xyz="0 0 -${leglen/2}" rpy="0 ${pi/2} 0"/> -->
         </collision>
-        <!-- <xacro:default_inertial mass="10"/> -->
+        <xacro:caster_inertial mass="${caster_mass}"/>
     </link>
     <joint name="base_link_to_${prefix}_caster" type="continuous">
@@ -53,5 +78,5 @@
         <child link="${prefix}_caster"/>
         <axis xyz="0 0 1"/>
-        <origin rpy="0 1.57075 0" xyz="0 -${0.2/2 + stem_lenght/2 + 0.1} ${reflect*(0.2/2 + 0.1)}"/>
+        <origin rpy="0 1.57075 0" xyz="0 -${body_x/2 + caster_radius*2} ${reflect*(body_z/2 + caster_radius)}"/>
     </joint>
     <joint name="base_link_to_${prefix}_caster_turn" type="continuous">
@@ -59,5 +84,5 @@
         <child link="${prefix}_caster"/>
         <axis xyz="1 0 0"/>
-        <origin rpy="0 1.57075 0" xyz="0 -${0.2/2 + stem_lenght/2 + 0.1} ${reflect*(0.2/2 + 0.1)}"/>
+        <origin rpy="0 1.57075 0" xyz="0 -${body_x/2 + caster_radius*2} ${reflect*(body_z/2 + caster_radius)}"/>
     </joint>
 </xacro:macro>
@@ -65,12 +90,13 @@
     <visual>
       <geometry>
-        <box size="0.8 1.5 0.2"/>
+        <box size="${body_x} ${body_y} ${body_z}"/>
       </geometry>
     </visual>
     <collision>
       <geometry>
-        <box size="0.8 1.5 0.2"/>
+        <box size="${body_x} ${body_y} ${body_z}"/>
       </geometry>
     </collision>
+    <xacro:caster_inertial mass="${body_mass}"/>
   </link>
 <xacro:wheel prefix="right" reflect="1" />

Commit message: URDF robot in Gazebo

File: diff_drive/urdf/ddrive.urdf.xacro (robot description, xacro)
@@ -16,5 +16,15 @@
 <xacro:property name="body_z"  value="${ros__parameters['body_z']}" />
 <xacro:property name="body_mass"  value="${ros__parameters['body_mass']}" />
-<xacro:property name="stem_lenght"  value="${platform_height-wheel_radius-wheel_radius-0.2-0.41-0.1}" />
+<xacro:include filename="$(find diff_drive)/ddrive.gazebo.xacro" />
+<material name = "red">
+    <color rgba ="1 0 0 1" />
+</material>
+<material name = "blue">
+    <color rgba ="0 0 1 1" />
+</material>
+<material name = "green">
+    <color rgba ="0 1 0 1" />
+</material>
+<!-- <link name="world"/>  -->
 <xacro:macro name="wheel_inertial" params="mass">
     <inertial>
@@ -33,5 +43,5 @@
     </inertial>
 </xacro:macro>
-<xacro:macro name="wheel" params="prefix reflect">
+<xacro:macro name="wheel" params="prefix reflect color">
     <link name="${prefix}_wheel">
         <visual>
@@ -39,4 +49,5 @@
                 <cylinder length="0.1" radius="0.3"/>
             </geometry>
+            <material name = "${color}" />
             <!-- <origin xyz="0 0 -${leglen/2}" rpy="0 ${pi/2} 0"/> -->
             <!-- <material name="white"/> -->
@@ -57,5 +68,5 @@
     </joint>
 </xacro:macro>
-<xacro:macro name="caster" params="prefix reflect">
+<xacro:macro name="caster" params="prefix reflect color">
     <link name="${prefix}_caster">
         <visual>
@@ -64,5 +75,5 @@
             </geometry>
             <!-- <origin xyz="0 0 -${leglen/2}" rpy="0 ${pi/2} 0"/> -->
-            <material name="white"/>
+            <material name = "${color}" />
         </visual>
         <collision>
@@ -74,10 +85,10 @@
         <xacro:caster_inertial mass="${caster_mass}"/>
     </link>
-    <joint name="base_link_to_${prefix}_caster" type="continuous">
+    <!-- <joint name="base_link_to_${prefix}_caster" type="continuous">
         <parent link="base_link"/>
         <child link="${prefix}_caster"/>
         <axis xyz="0 0 1"/>
         <origin rpy="0 1.57075 0" xyz="0 -${body_x/2 + caster_radius*2} ${reflect*(body_z/2 + caster_radius)}"/>
-    </joint>
+    </joint> -->
     <joint name="base_link_to_${prefix}_caster_turn" type="continuous">
         <parent link="base_link"/>
@@ -92,4 +103,5 @@
         <box size="${body_x} ${body_y} ${body_z}"/>
       </geometry>
+      <material name = "red" />
     </visual>
     <collision>
@@ -100,7 +112,7 @@
     <xacro:caster_inertial mass="${body_mass}"/>
   </link>
-<xacro:wheel prefix="right" reflect="1" />
-<xacro:wheel prefix="left" reflect="-1" />
-<xacro:caster prefix="top" reflect="1" />
-<xacro:caster prefix="bottom" reflect="-1" />
+<xacro:wheel prefix="right" reflect="1" color ="blue"/>
+<xacro:wheel prefix="left" reflect="-1" color ="blue"/>
+<xacro:caster prefix="top" reflect="1" color ="green"/>
+<xacro:caster prefix="bottom" reflect="-1" color ="green"/>
 </robot>

Commit message: Took out models from .world and car now falls

File: diff_drive/urdf/ddrive.urdf.xacro (robot description, xacro)
@@ -72,5 +72,6 @@
         <visual>
             <geometry>
-                <cylinder length="0.1" radius="0.1"/>
+                <!-- <cylinder length="0.1" radius="0.1"/> -->
+                <sphere radius="${caster_radius}"/>
             </geometry>
             <!-- <origin xyz="0 0 -${leglen/2}" rpy="0 ${pi/2} 0"/> -->
@@ -79,5 +80,6 @@
         <collision>
             <geometry>
-                <cylinder length="${caster_length}" radius="${caster_radius}"/>
+                <!-- <cylinder length="${caster_length}" radius="${caster_radius}"/> -->
+                <sphere radius="${caster_radius}"/>
             </geometry>
             <!-- <origin xyz="0 0 -${leglen/2}" rpy="0 ${pi/2} 0"/> -->

Commit message: Added inertial calculations

File: diff_drive/urdf/ddrive.urdf.xacro (robot description, xacro)
@@ -10,5 +10,4 @@
 <xacro:property name="wheel_mass"  value="${ros__parameters['wheel_mass']}" />
 <xacro:property name="caster_radius"  value="${ros__parameters['caster_radius']}" />
-<xacro:property name="caster_length"  value="${ros__parameters['caster_length']}" />
 <xacro:property name="caster_mass"  value="${ros__parameters['caster_mass']}" />
 <xacro:property name="body_x"  value="${ros__parameters['body_x']}" />
@@ -29,7 +28,7 @@
     <inertial>
             <mass value="${mass}" />
-            <inertia ixx="1e-3" ixy="0.0" ixz="0.0"
-                 iyy="1e-3" iyz="0.0"
-                 izz="1e-3" />
+            <inertia ixx="${mass*(3*wheel_radius**2 + wheel_length**2)/12}" ixy="0.0" ixz="0.0"
+                 iyy="${mass*(3*wheel_radius**2 + wheel_length**2)/12}" iyz="0.0"
+                 izz="${mass*(wheel_radius**2)/2}" />
     </inertial>
 </xacro:macro>
@@ -37,7 +36,15 @@
     <inertial>
             <mass value="${mass}" />
-            <inertia ixx="1e-3" ixy="0.0" ixz="0.0"
-                 iyy="1e-3" iyz="0.0"
-                 izz="1e-3" />
+            <inertia ixx="${mass*(caster_radius**2 + caster_radius**2)/5}" ixy="0.0" ixz="0.0"
+                 iyy="${mass*(caster_radius**2 + caster_radius**2)/5}" iyz="0.0"
+                 izz="${mass*(caster_radius**2 + caster_radius**2)/5}"/>
+    </inertial>
+</xacro:macro>
+<xacro:macro name="body_inertial" params="mass">
+    <inertial>
+            <mass value="${mass}" />
+            <inertia ixx="${mass*(body_y**2 + body_z**2)/12}" ixy="0.0" ixz="0.0"
+                 iyy="${mass*(body_x**2 + body_z**2)/12}" iyz="0.0"
+                 izz="${mass*(body_x**2 + body_y**2)/12}" />
     </inertial>
 </xacro:macro>
@@ -98,5 +105,5 @@
       </geometry>
     </collision>
-    <xacro:caster_inertial mass="${body_mass}"/>
+    <xacro:body_inertial mass="${body_mass}"/>
   </link>
 <xacro:wheel prefix="right" reflect="1" color ="blue"/>

Commit message: Done just add doc strings

File: diff_drive/urdf/ddrive.urdf.xacro (robot description, xacro)
@@ -5,5 +5,4 @@
 <xacro:property name="start"  value="${props['/**']}" />
 <xacro:property name="ros__parameters"  value="${start['ros__parameters']}" />
-<xacro:property name="platform_height"  value="${ros__parameters['platform_height']}" />
 <xacro:property name="wheel_radius"  value="${ros__parameters['wheel_radius']}" />
 <xacro:property name="wheel_length"  value="${ros__parameters['wheel_length']}" />
